Commit message: sim: migrate to Gazebo Harmonic and make the sim stack runnable on Jazzy
Local work from 2026-09-12 to 2026-10-08 that never reached the repo:

- Gazebo Classic -> Harmonic: ros_gz_sim gz_sim.launch.py + create instead of
  gazebo_ros/spawn_entity.py, ros_gz_bridge parameter_bridge, gpu_lidar /
  depth_camera / camera sensors with gz_frame_id, gz_ros2_control
  (launch_sim, docking_sim, sim_nav, sim_mapping, xacros, worlds,
  my_sim_controllers, package.xml).
- GZ_IP=127.0.0.1 default in the sim launches (gz discovery over loopback;
  the dev host filters multicast on its NIC), gz_headless arg.
- turtlebot3_house / turtlebot3_world worlds + models (installed via CMake).
- stvl_sim_params: collision_monitor section (Nav2 bringup aborted without
  it), AMCL retune for slip-free sim odometry, STVL disabled in the sim.
- nevo_diagnostic_node: enable_stack_lock param so launch_sim + sim_nav can
  run as one session.
- IMU sketch for the ESP8266 + MPU6050 (Wire.begin(4, 0)).
- config_nevo.rviz updates, uncommitted session reports.

Co-Authored-By: Claude Opus 5.5 <noreply@anthropic.com>

File: src/nevo-dev/nevo_bot/description/c310_camera.xacro (robot description, xacro)
@@ -31,13 +31,23 @@
     </joint>
     <link name="c310_camera_link_optical"></link>
+    <!--
+      Gazebo Harmonic: Classic libgazebo_ros_camera.so replaced by a native
+      camera sensor. Topic c310/image_raw makes gz publish
+        /c310/image_raw     image (bridged to ROS 1:1)
+        /c310/camera_info   derived from the topic's parent path
+      which is exactly what the AprilTag docking pipeline subscribes to.
+    -->
     <gazebo reference="c310_camera_link">
         <sensor name="c310_camera" type="camera">
             <pose>0 0 0 0 0 0</pose>
             <visualize>false</visualize>
-            <update_rate>15</update_rate>
+            <always_on>true</always_on>
+            <update_rate>5</update_rate>
+            <topic>c310/image_raw</topic>
+            <gz_frame_id>c310_camera_link_optical</gz_frame_id>
             <camera>
                 <horizontal_fov>1.089</horizontal_fov>
                 <image>
-                    <format>B8G8R8</format>
+                    <format>R8G8B8</format>
                     <width>640</width>
                     <height>480</height>
@@ -48,11 +58,4 @@
                 </clip>
             </camera>
-            <plugin name="c310_camera_controller" filename="libgazebo_ros_camera.so">
-                <frame_name>c310_camera_link_optical</frame_name>
-                <ros>
-                    <argument>camera_info:=/c310/camera_info</argument>
-                    <argument>image_raw:=/c310/image_raw</argument>
-                </ros>
-            </plugin>
         </sensor>
     </gazebo>

File: src/nevo-dev/nevo_bot/description/depth_camera.xacro (robot description, xacro)
@@ -25,14 +25,30 @@
     </joint>
     <link name="camera_link_optical"></link>
+    <!--
+      Gazebo Harmonic: Classic libgazebo_ros_camera.so replaced by a native
+      depth_camera sensor. gz topics produced:
+        /camera/depth/image_raw       depth image (32FC1 once bridged)
+        /camera/depth/camera_info     derived from the topic's parent path
+        /camera/depth/image_raw/points  point cloud (bridged to /camera/points)
+    -->
     <gazebo reference="camera_link">
-        <material>Gazebo/Red</material>
-        <sensor name="camera" type="depth">
-            <pose> 0 0 0 0 0 0 </pose>
+        <visual>
+            <material>
+                <ambient>1 0 0 1</ambient>
+                <diffuse>1 0 0 1</diffuse>
+                <specular>0.5 0.5 0.5 1</specular>
+            </material>
+        </visual>
+        <sensor name="camera" type="depth_camera">
+            <pose>0 0 0 0 0 0</pose>
             <visualize>true</visualize>
-            <update_rate>10</update_rate>
+            <always_on>true</always_on>
+            <update_rate>5</update_rate>
+            <topic>camera/depth/image_raw</topic>
+            <gz_frame_id>camera_link_optical</gz_frame_id>
             <camera>
                 <horizontal_fov>1.089</horizontal_fov>
                 <image>
-                    <format>B8G8R8</format>
+                    <format>R8G8B8</format>
                     <width>640</width>
                     <height>480</height>
@@ -43,9 +59,4 @@
                 </clip>
             </camera>
-            <plugin name="camera_controller" filename="libgazebo_ros_camera.so">
-                <frame_name>camera_link_optical</frame_name>
-                <min_depth>0.1</min_depth>
-                <max_depth>100.0</max_depth>
-            </plugin>
         </sensor>
     </gazebo>

File: src/nevo-dev/nevo_bot/description/lidar.xacro (robot description, xacro)
@@ -22,14 +22,29 @@
         </xacro:inertial_cylinder>
     </link>
+    <!--
+      Gazebo Harmonic: the Classic libgazebo_ros_ray_sensor.so plugin does not
+      exist here. The gpu_lidar sensor publishes on gz topic /scan with the
+      frame stamped by <gz_frame_id>; launch_sim.launch.py bridges it to ROS.
+    -->
     <gazebo reference="laser_frame">
-        <material>Gazebo/Black</material>
-        <sensor name="laser" type="ray">
-            <pose> 0 0 0 0 0 0 </pose>
+        <visual>
+            <material>
+                <ambient>0.1 0.1 0.1 1</ambient>
+                <diffuse>0.1 0.1 0.1 1</diffuse>
+                <specular>0.2 0.2 0.2 1</specular>
+            </material>
+        </visual>
+        <sensor name="laser" type="gpu_lidar">
+            <pose>0 0 0 0 0 0</pose>
             <visualize>false</visualize>
+            <always_on>true</always_on>
             <update_rate>10</update_rate>
-            <ray>
+            <topic>scan</topic>
+            <gz_frame_id>laser_frame</gz_frame_id>
+            <lidar>
                 <scan>
                     <horizontal>
                         <samples>360</samples>
+                        <resolution>1</resolution>
                         <min_angle>-3.14</min_angle>
                         <max_angle>3.14</max_angle>
@@ -39,13 +54,7 @@
                     <min>0.3</min>
                     <max>12</max>
+                    <resolution>0.01</resolution>
                 </range>
-            </ray>
-            <plugin name="laser_controller" filename="libgazebo_ros_ray_sensor.so">
-                <ros>
-                    <argument>~/out:=scan</argument>
-                </ros>
-                <output_type>sensor_msgs/LaserScan</output_type>
-                <frame_name>laser_frame</frame_name>
-            </plugin>
+            </lidar>
         </sensor>
     </gazebo>

File: src/nevo-dev/nevo_bot/description/ros2_control_sim.xacro (robot description, xacro)
@@ -1,7 +1,13 @@
 <?xml version="1.0"?>
 <robot xmlns:xacro="http://www.ros.org/wiki/xacro">
-    <ros2_control name="GazeboSystem" type="system">
+    <!--
+      Gazebo Harmonic (gz-sim) simulation hardware, replaces the Gazebo Classic
+      gazebo_ros2_control/GazeboSystem that is unavailable on ROS 2 Jazzy.
+      The gz-sim system plugin below is what starts ros2_control's
+      controller_manager inside the simulation process.
+    -->
+    <ros2_control name="GazeboSimSystem" type="system">
         <hardware>
-            <plugin>gazebo_ros2_control/GazeboSystem</plugin>
+            <plugin>gz_ros2_control/GazeboSimSystem</plugin>
         </hardware>
         <joint name="left_wheel_joint">
@@ -23,5 +29,5 @@
     </ros2_control>
     <gazebo>
-        <plugin name="gazebo_ros2_control" filename="libgazebo_ros2_control.so">
+        <plugin filename="gz_ros2_control-system" name="gz_ros2_control::GazeboSimROS2ControlPlugin">
             <parameters>$(find nevo_bot)/config/my_sim_controllers.yaml</parameters>
         </plugin>
