Commit message: update: imu sensor fusion

File: src/nevo-dev/nevo_bot/description/robot_core.xacro (robot description, xacro)
@@ -18,12 +18,12 @@
         <color rgba="1 0 0 1"/>
     </material>
+    <link name="base_link">
+    </link>
+    <joint name="base_footprint_joint" type="fixed">
+        <parent link="base_link"/>
+        <child link="base_footprint"/>
+        <origin xyz="0 0 0" rpy="0 0 0"/>
+    </joint>
     <link name="base_footprint">
-    </link>
-    <joint name="base_footprint_joint" type="fixed">
-        <parent link="base_footprint"/>
-        <child link="base_link"/>
-        <origin xyz="0 0 0" rpy="0 0 0"/>
-    </joint>
-    <link name="base_link">
     </link>
     <joint name="chassis_joint" type="fixed">

Commit message: hw: track the active map on MAP_SELECTED; URDF wheel separation 0.425 m

File: src/nevo-dev/nevo_bot/description/robot_core.xacro (robot description, xacro)
@@ -62,5 +62,5 @@
         <parent link="base_link"/>
         <child link="left_wheel"/>
-        <origin xyz="0.0 0.26 0.0635" rpy="-${pi/2} 0 0"/>
+        <origin xyz="0.0 0.2125 0.0635" rpy="-${pi/2} 0 0"/>  <!-- wheel_separation 0.425 m (measured 42 cm), same as diff_cont -->
         <axis xyz="0.0 0.0 1.0"/>
     </joint>
@@ -102,5 +102,5 @@
         <parent link="base_link"/>
         <child link="right_wheel"/>
-        <origin xyz="0.0 -0.26 0.0635" rpy="${pi/2} 0 0"/>
+        <origin xyz="0.0 -0.2125 0.0635" rpy="${pi/2} 0 0"/>
         <axis xyz="0.0 0.0 -1.0"/>
     </joint>
