Commit message: hw: IMU and Kinect calibration, mapping with Nav2, thesis nav configs
- IMU (re-soldered Nano + new GY-521): mount_up [0.0962, -0.0458, 0.9943], gyro_scale_z
  1.0023 set in launch_robot (lidar-ICP calibrated; EKF heading ~0.2 % over 3 turns)
- Kinect camera_joint xyz 0.495 0 1.0, rpy 0 0.0428 0.035 (lab + wall calibration);
  kinect_ros2 full_depth_every_n (launch: 3 -> full depth 10 Hz, /points stays 30 Hz)
- launch_robot nav:=true in mapping mode starts Nav2 with the stock BT; slam_pose_correction
  re-anchors slam_toolbox from an RViz 2D Pose Estimate
- hw_nav_dwb/mppi: xy_goal_tolerance 0.15 (pass criterion stays +-0.20 m)

Co-Authored-By: Claude Opus 5.5 <noreply@anthropic.com>

File: src/nevo-dev/nevo_bot/description/depth_camera.xacro (robot description, xacro)
@@ -4,5 +4,12 @@
         <parent link="chassis"/>
         <child link="camera_link"/>
-        <origin xyz="0.46 0 1.0" rpy="0 0 0"/>
+        <!-- Calibrated 2026-10-25 (lab + wall bags, see src/scripts/cafe_survey):
+             x 0.495: lidar centre -> Kinect face measured ~19.5 cm (was 0.46).
+             pitch 0.0428 rad = 2.45 deg down: mostly the whole body leaning on the
+               lower front caster, so it varies 1-3 deg with how the robot settles.
+             yaw 0.035 rad = 2.0 deg left of the lidar (wall seen by both sensors).
+             Height 0.99 m and roll -0.27 deg measured, left as is.
+             The Kinect has a tilt motor: re-check after it has been moved. -->
+        <origin xyz="0.495 0 1.0" rpy="0 0.0428 0.035"/>
     </joint>
     <link name="camera_link">
